File: _autosave-SIN-PAD.kicad_pcb (KiCad board)
At the start: 2 copper layers, 56 parts, among them SW1 SW_Push, U1 ATmega32U4-AU, Y1 16MHz

Commit message: Nyt alkaa muodostuu
Parts:
- removed C1, C2: 22pF, Capacitor_SMD:C_0805_2012Metric
- removed C3: 1uf, Capacitor_SMD:C_0805_2012Metric
- removed C4, C5, C6: 0.1uF, Capacitor_SMD:C_0805_2012Metric
- removed C7: 10uF, Capacitor_SMD:C_0805_2012Metric
- removed F1: 500mA, Fuse:Fuse_1206_3216Metric
- removed MX1: MX-NoLED, MX_Only:MXOnly-1U-NoLED
- removed R1, R4: 10k, Resistor_SMD:R_0805_2012Metric
- removed R2, R3: 22, Resistor_SMD:R_0805_2012Metric
- removed SW1: SW_Push, random-keyboard-parts:SKQG-1155865
- removed USB1: Molex-0548190589, random-keyboard-parts:Molex-0548190589
- removed Y1: 16MHz, Crystal:Crystal_SMD_3225-4Pin_3.2x2.5mm
- added J1: Connector COL, Connector_PinHeader_2.00mm:PinHeader_1x01_P2.00mm_Vertical, F.Cu at (47.6, 90.5)
- added J2: Conn_01x01_Female, Connector_PinHeader_2.00mm:PinHeader_1x01_P2.00mm_Vertical, F.Cu at (33.3, 92.9)
- D1, D10, D11, D12, D13, D14, D15, D16, D17, D18, D19, D2, D20, D3, D4, D5, D6, D7, D8, D9: footprint Diode_SMD:D_SOD-123 -> Keebio-Parts:Diode-Hybrid-Back
- U1: value ATmega32U4-AU -> ProMicro; footprint Package_QFP:TQFP-44_10x10mm_P0.8mm -> Keebio-Parts:ArduinoProMicro
- moved U1 61.2 mm to (159.5, 35.7)
- moved D16 52.2 mm to (73.8, 142.9), turned to 270 degrees
- moved D20 52.2 mm to (73.8, 161.9), turned to 270 degrees
- moved D9 52.2 mm to (73.8, 114.3), turned to 270 degrees
- moved D2 51.9 mm to (54.8, 61.9), turned to 270 degrees
- moved D3 51.9 mm to (73.8, 61.9), turned to 270 degrees
- moved D4 51.9 mm to (54.8, 81.0), turned to 270 degrees
- moved D5 51.9 mm to (73.8, 81.0), turned to 270 degrees
- moved MX16 34.0 mm to (83.3, 142.9)
- moved MX20 34.0 mm to (83.3, 161.9)
- moved MX9 33.9 mm to (83.3, 114.3), turned to 270 degrees
- moved MX2 33.5 mm to (64.3, 61.9)
- moved MX3 33.5 mm to (83.3, 61.9)
- moved MX4 33.5 mm to (64.3, 81.0)
- moved MX5 33.5 mm to (83.3, 81.0)
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Connections:
- D1 pad 1: ROW0 -> ROW2
- U1 pad 14: +5V -> Net-(U1-Pad14)
- U1 pad 15: GND -> Net-(U1-Pad15)
- U1 pad 2: +5V -> Net-(U1-Pad2)
- U1 pad 23: GND -> Net-(U1-Pad23)
- U1 pad 24: +5V -> Net-(U1-Pad24)
- U1 pad 5: GND -> Net-(U1-Pad5)
- U1 pad 7: +5V -> Net-(U1-Pad7)
