File: SIN-PAD.kicad_pcb (KiCad board)
At the start: 2 copper layers, 42 parts, among them J1 Connector COL, J2 Conn_01x01_Female, U1 ProMicro

Commit message: Muutamii muutoksia
Parts:
- added   : LOGO, Keepoprints:pikkunimmari, B.Cu at (96.4, 67.0)
- added G***: LOGO, Keepoprints:bcsmol, F.Cu at (82.2, 106.0)
- added G***: LOGO, Keepoprints:kaffe, B.Cu at (111.9, 101.2)
- added G***: LOGO, Keepoprints:meitsinormi, B.Cu at (81.0, 98.0)
- J1, J2: footprint Connector_PinHeader_2.00mm:PinHeader_1x01_P2.00mm_Vertical -> Connector_Wire:SolderWire-0.5sqmm_1x01_D0.9mm_OD2.3mm
- moved J1 46.7 mm to (117.9, 70.2)
- moved J2 46.7 mm to (113.1, 70.2), turned to 180 degrees
- moved D2 43.3 mm to (103.6, 35.7)
- moved D4 43.3 mm to (103.6, 54.8)
- moved D5 39.6 mm to (114.3, 64.3), turned to 180 degrees
- moved D3 39.5 mm to (114.1, 45.2), turned to 180 degrees
- moved D1 26.6 mm to (104.8, 66.7), turned to 180 degrees
- moved MX10 24.5 mm to (50.0, 97.6)
- moved MX11 24.5 mm to (69.1, 97.6)
- moved MX12 24.5 mm to (88.1, 97.6)
- moved MX13 24.5 mm to (50.0, 116.7)
- moved MX14 24.5 mm to (69.1, 116.7)
- moved MX15 24.5 mm to (88.1, 116.7)
- moved MX16 24.5 mm to (111.9, 116.7)
- moved MX2 24.5 mm to (92.9, 35.7)
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Connections:
- U1 pad 1: Net-(U1-Pad1) -> unconnected-(U1-Pad1)
- U1 pad 10: Net-(U1-Pad10) -> COL2
- U1 pad 11: Net-(U1-Pad11) -> unconnected-(U1-Pad11)
- U1 pad 12: Net-(U1-Pad12) -> unconnected-(U1-Pad12)
- U1 pad 13: Net-(U1-Pad13) -> ROW2
- U1 pad 14: Net-(U1-Pad14) -> COL3
- U1 pad 15: Net-(U1-Pad15) -> ROW5
- U1 pad 16: Net-(U1-Pad16) -> ROW4
- U1 pad 17: Net-(U1-Pad17) -> ROW3
- U1 pad 18: Net-(U1-Pad18) -> unconnected-(U1-Pad18)
- U1 pad 19: Net-(U1-Pad19) -> ROW1
- U1 pad 2: Net-(U1-Pad2) -> unconnected-(U1-Pad2)
- U1 pad 20: Net-(U1-Pad20) -> ROW0
- U1 pad 21: Net-(U1-Pad21) -> unconnected-(U1-Pad21)
- U1 pad 22: Net-(U1-Pad22) -> unconnected-(U1-Pad22)
- U1 pad 23: Net-(U1-Pad23) -> unconnected-(U1-Pad23)
- U1 pad 24: Net-(U1-Pad24) -> unconnected-(U1-Pad24)
- U1 pad 3: Net-(U1-Pad3) -> unconnected-(U1-Pad3)
- U1 pad 4: Net-(U1-Pad4) -> unconnected-(U1-Pad4)
- U1 pad 5: Net-(U1-Pad5) -> unconnected-(U1-Pad5)
- U1 pad 6: Net-(U1-Pad6) -> unconnected-(U1-Pad6)
- U1 pad 7: Net-(U1-Pad7) -> unconnected-(U1-Pad7)
- U1 pad 8: Net-(U1-Pad8) -> COL0
- U1 pad 9: Net-(U1-Pad9) -> COL1
Routing:
- net ROW5: track 0.00 -> 137.2 mm
- net COL0: track 0.00 -> 122.2 mm
- net ROW4: track 0.00 -> 119.0 mm
- net COL3: track 0.00 -> 116.6 mm
- net ROW3: track 0.00 -> 107.6 mm
- net COL2: track 0.00 -> 106.0 mm
- net COL1: track 0.00 -> 100.5 mm
- net ROW2: track 0.00 -> 65.3 mm
- net ROW1: track 0.00 -> 28.8 mm
- net Net-(D5-Pad2): track 0.00 -> 18.7 mm
- net Net-(D9-Pad2): track 0.00 -> 18.1 mm
- net Net-(D3-Pad2): track 0.00 -> 18.1 mm
- net ROW0: track 0.00 -> 12.8 mm
- net Net-(D20-Pad2): track 0.00 -> 12.6 mm
- net Net-(D16-Pad2): track 0.00 -> 12.6 mm
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Other:
- board outline added: 78.6 x 116.7 mm
- net class Default removed
